File: Драйвер IGBT/Драйвер IGBT.kicad_pcb (KiCad board)
At the start: 4 copper layers, 142.2 x 68.6 mm, 41 parts, among them J1 DC+, J2 DC-, J3 Control Connector, J4 OUT-, J5 OUT+, Q1 HGTG20N60A4, U3 L78L05ACUTR

Commit message: VER2.0
Parts:
- removed D7: LED_FLT, LED_SMD:LED_0603_1608Metric_Pad1.05x0.95mm_HandSolder
- removed U3: L78L05ACUTR, Package_TO_SOT_SMD:SOT-89-3
- added R8: 10k, Resistor_SMD:R_0805_2012Metric_Pad1.15x1.40mm_HandSolder, F.Cu at (166.7, 74.2)
- added R9: 10k, Resistor_SMD:R_0805_2012Metric_Pad1.15x1.40mm_HandSolder, F.Cu at (166.9, 76.5)
- added U1: LM1117-ADJ, Package_TO_SOT_SMD:SOT-223, F.Cu at (148.2, 84.0)
- C17: value 0.33u -> 10u
- C18: value 0.1u -> 10u
- D1: value VS-60APU06PBF -> VS-60EPF06-M3; footprint Package_TO_SOT_THT:TO-247-3_Vertical -> Package_TO_SOT_THT:TO-247-2_Vertical
- D3: value PDZ6.2BGWX -> MMSZ5223B
- D5: value D_Small -> MURS360T3G
- D8: footprint Converter_DCDC:Converter_DCDC_TRACO_TMR-1-xxxx_Dual_THT -> TRACO:TMA1515S
- R4: value 1.1k -> 6.8k
- moved R7 36.9 mm to (172.9, 79.5)
- moved C6 35.1 mm to (139.3, 83.9), turned to 90 degrees
- moved D8 27.2 mm to (135.5, 81.6), turned to 270 degrees
- moved R1 26.3 mm to (159.6, 77.8), turned to 0 degrees
- moved D3 25.9 mm to (177.8, 96.9)
- moved C10 25.9 mm to (172.8, 96.9)
- moved C9 25.9 mm to (170.8, 96.9)
- moved D4 25.9 mm to (175.2, 96.9)
- moved D5 25.0 mm to (175.2, 87.3), turned to 270 degrees
- moved C7 24.9 mm to (159.7, 80.0), turned to 180 degrees
- moved C2 24.9 mm to (139.3, 75.0), turned to 270 degrees
- moved R5 24.3 mm to (166.5, 96.8)
- moved R4 24.3 mm to (160.9, 96.8)
- moved R6 24.3 mm to (163.5, 96.8)
- moved D2 23.8 mm to (164.2, 87.2)
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Connections:
- C1 pad 1: D_IGBT -> DC+
- C10 pad 2: OUT+ -> DC-
- C11 pad 1: D_IGBT -> DC+
- C4 pad 1: D_IGBT -> DC+
- C5 pad 1: D_IGBT -> DC+
- C6 pad 2: OUT+ -> DC-
- C8 pad 1: D_IGBT -> DC+
- C9 pad 2: OUT+ -> DC-
- D1 pad 1: DC- -> DC+
- D1 pad 2: OUT+ -> D_IGBT
- D2 pad 1: OUT+ -> DC-
- D2 pad 3: OUT+ -> DC-
- D2 pad 7: (no net) -> G_IGBT
- D2 pad 8: OUT+ -> DC-
- D4 pad 2: OUT+ -> DC-
- D6 pad 5: DC- -> D_IGBT
- D6 pad 6: DC- -> D_IGBT
- D6 pad 7: DC- -> D_IGBT
- D6 pad 8: DC- -> D_IGBT
- D8 pad 4: OUT+ -> DC-
- J1 pad 1: D_IGBT -> DC+
- J1 pad 2: D_IGBT -> DC+
- J1 pad 3: D_IGBT -> DC+
- J1 pad 4: D_IGBT -> DC+
- J1 pad 5: D_IGBT -> DC+
- J1 pad 6: D_IGBT -> DC+
- J1 pad 7: D_IGBT -> DC+
- J1 pad 8: D_IGBT -> DC+
- J3 pad 1: RDY -> +15V
- J3 pad 2: FLT -> Measure
- J3 pad 3: RST -> IN-
- J3 pad 4: GNDA -> IN+
- J3 pad 5: IN- -> GNDA
- J3 pad 6: IN+ -> RST
- J3 pad 7: Measure -> FLT
- J3 pad 8: +15V -> RDY
- J5 pad 1: OUT+ -> DC+
- J5 pad 2: OUT+ -> DC+
- J5 pad 3: OUT+ -> DC+
- J5 pad 4: OUT+ -> DC+
- J5 pad 5: OUT+ -> DC+
- J5 pad 6: OUT+ -> DC+
- J5 pad 7: OUT+ -> DC+
- J5 pad 8: OUT+ -> DC+
- Q1 pad 3: OUT+ -> DC-
- R2 pad 2: OUT+ -> DC-
Routing:
- net OUT+: track 98.7 -> 0.00 mm, vias 92 -> 0
- net GNDA: track 133.3 -> 45.1 mm, vias 3 -> 4
- net +5V: track 74.5 -> 10.4 mm, vias 2 -> 3
- net DC-: track 6.16 -> 60.0 mm, vias 76 -> 5
- net D_IGBT: track 62.1 -> 13.8 mm, vias 35 -> 0
- net G_IGBT: track 42.2 -> 20.6 mm, vias 1 -> 0
- net FLT: track 37.1 -> 18.7 mm, vias 2 -> 1
- net RST: track 24.4 -> 17.4 mm
- net Desat: track 22.1 -> 28.9 mm, vias 3 -> 2
- net IN+: track 11.9 -> 18.2 mm, vias 0 -> 1
- net IN-: track 21.3 -> 27.6 mm, vias 2 -> 1
- net Net-(D3-Pad2): track 12.9 -> 6.96 mm
- net Measure: track 41.2 -> 46.2 mm
- net +15V_H: track 62.4 -> 59.0 mm
- net Vcc: track 7.98 -> 4.92 mm
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- added copper zone on In2.Cu, net +5V
- added copper zone on F.Cu, net DC+
- added copper zone on In2.Cu, net DC+
- added copper zone on B.Cu, net D_IGBT
- added copper zone on In1.Cu, net GNDA
- added copper zone on F.Cu, net G_IGBT
- removed copper zone on F.Cu, net D_IGBT
- removed copper zone on B.Cu, net OUT+
- removed copper zone on In2.Cu, net OUT+

Commit message: VER2.2
Parts:
- moved D5 20.8 mm to (177.6, 108.0), turned to 90 degrees
Routing:
- net +15V_H: track 59.0 -> 7.72 mm
- net DC-: track 60.0 -> 47.8 mm
- net Net-(D3-Pad2): track 6.96 -> 13.1 mm
- net D_IGBT: track 13.8 -> 16.8 mm
- added copper zone on In2.Cu, net +15V_H
- added copper zone on In1.Cu, net DC-

Commit message: VER2.2
Parts:
- moved C17 3.30 mm to (154.2, 77.4)
- moved C18 3.30 mm to (154.2, 81.9)
- moved U1 3.30 mm to (148.2, 80.7)
Routing:
- net +15V: track 31.9 -> 29.1 mm
- net GNDA: track 45.1 -> 47.5 mm
Changed lines of the file:
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@@
     (thickness 1.6)
     (drawings 25)
-    (tracks 192)
+    (tracks 194)
     (zones 0)
     (modules 42)
@@
   )
   (module Package_TO_SOT_SMD:SOT-223 (layer F.Cu)
-    (at 148.1823 84.0256 180)
+    (at 148.1823 80.7236 180)
     (descr "module CMS SOT223 4 pins")
     (tags "CMS SOT")
@@
   )
   (module Capacitor_SMD:C_0805_2012Metric_Pad1.15x1.40mm_HandSolder (layer F.Cu)
-    (at 154.1513 85.1596 270)
+    (at 154.1513 81.8576 270)
     (descr "Capacitor SMD 0805 (2012 Metric), square (rectangular) end terminal, IPC_7351 nominal with elongated pad for handsoldering. (Body size source: https://docs.google.com/spreadsheets/d/1BsfQQcO9C6DZCsRaXUlFlo91Tg2WpOkGARC1WS5S8t0/edit?usp=sharing), generated with kicad-footprint-generator")
     (tags "capacitor handsolder")
@@
   )
   (module Capacitor_SMD:C_0805_2012Metric_Pad1.15x1.40mm_HandSolder (layer F.Cu)
-    (at 154.1513 80.7236 90)
+    (at 154.1513 77.4216 90)
     (descr "Capacitor SMD 0805 (2012 Metric), square (rectangular) end terminal, IPC_7351 nominal with elongated pad for handsoldering. (Body size source: https://docs.google.com/spreadsheets/d/1BsfQQcO9C6DZCsRaXUlFlo91Tg2WpOkGARC1WS5S8t0/edit?usp=sharing), generated with kicad-footprint-generator")
     (tags "capacitor handsolder")
@@
   (segment (start 166.0893 91.8506) (end 166.0893 94.8571) (width 0.5) (layer F.Cu) (net 5))
   (segment (start 163.5493 91.8506) (end 163.5493 95.3016) (width 0.5) (layer F.Cu) (net 6))
-  (segment (start 154.0423 84.0256) (end 154.1513 84.1346) (width 1) (layer F.Cu) (net 7))
-  (segment (start 151.3323 84.0256) (end 154.0423 84.0256) (width 1) (layer F.Cu) (net 7))
-  (segment (start 154.1513 84.1346) (end 156.1653 84.1346) (width 0.5) (layer F.Cu) (net 7))
-  (segment (start 156.1653 84.1346) (end 156.1653 84.1346) (width 0.5) (layer F.Cu) (net 7))
-  (via (at 156.1653 84.1346) (size 0.8) (drill 0.4) (layers F.Cu B.Cu) (net 7))
+  (segment (start 154.0423 80.7236) (end 154.1513 80.8326) (width 1) (layer F.Cu) (net 7))
+  (segment (start 151.3323 80.7236) (end 154.0423 80.7236) (width 1) (layer F.Cu) (net 7))
+  (via (at 155.6753 80.8506) (size 0.8) (drill 0.4) (layers F.Cu B.Cu) (net 7))
   (segment (start 158.5873 77.8026) (end 156.9453 77.8026) (width 0.5) (layer F.Cu) (net 7))
   (segment (start 156.9453 77.8026) (end 156.9453 77.8026) (width 0.5) (layer F.Cu) (net 7))
@@
   (segment (start 192.7593 77.5486) (end 194.4193 75.8886) (width 0.5) (layer F.Cu) (net 13))
   (segment (start 192.7593 78.8086) (end 192.7593 80.7136) (width 0.5) (layer F.Cu) (net 13))
-  (segment (start 154.0103 86.3256) (end 154.1513 86.1846) (width 1) (layer F.Cu) (net 13))
-  (segment (start 151.3323 86.3256) (end 154.0103 86.3256) (width 1) (layer F.Cu) (net 13))
+  (segment (start 154.0103 83.0236) (end 154.1513 82.8826) (width 1) (layer F.Cu) (net 13))
+  (segment (start 151.3323 83.0236) (end 154.0103 83.0236) (width 1) (layer F.Cu) (net 13))
   (segment (start 159.7393 80.8366) (end 158.8643 79.9616) (width 0.5) (layer F.Cu) (net 13))
   (segment (start 159.7393 82.5506) (end 159.7393 80.8366) (width 0.5) (layer F.Cu) (net 13))
@@
   (segment (start 156.9453 79.9616) (end 156.9453 79.9616) (width 0.5) (layer F.Cu) (net 13))
   (via (at 156.9453 79.9616) (size 0.8) (drill 0.4) (layers F.Cu B.Cu) (net 13))
-  (segment (start 156.6823 79.6986) (end 156.9453 79.9616) (width 0.5) (layer F.Cu) (net 13))
-  (segment (start 154.1513 79.6986) (end 156.6823 79.6986) (width 0.5) (layer F.Cu) (net 13))
-  (segment (start 151.3323 86.3256) (end 148.3233 86.3256) (width 0.5) (layer F.Cu) (net 13))
-  (segment (start 148.3233 86.3256) (end 148.3233 86.3256) (width 0.5) (layer F.Cu) (net 13))
-  (via (at 148.3233 86.3256) (size 0.8) (drill 0.4) (layers F.Cu B.Cu) (net 13))
+  (segment (start 151.3323 83.0236) (end 148.3233 83.0236) (width 0.5) (layer F.Cu) (net 13))
+  (segment (start 148.3233 83.0236) (end 148.3233 83.0236) (width 0.5) (layer F.Cu) (net 13))
+  (via (at 148.3233 83.0236) (size 0.8) (drill 0.4) (layers F.Cu B.Cu) (net 13))
   (segment (start 139.2558 76.5326) (end 139.2923 76.4961) (width 1) (layer F.Cu) (net 13))
   (segment (start 135.4823 76.5326) (end 139.2558 76.5326) (width 1) (layer F.Cu) (net 13))
@@
   (segment (start 141.9228 76.4961) (end 146.0118 76.4961) (width 1) (layer B.Cu) (net 13))
   (segment (start 146.5073 76.0006) (end 151.4843 71.0236) (width 1) (layer B.Cu) (net 13))
-  (segment (start 154.1283 81.7256) (end 154.1513 81.7486) (width 1) (layer F.Cu) (net 14))
-  (segment (start 151.3323 81.7256) (end 154.1283 81.7256) (width 1) (layer F.Cu) (net 14))
+  (segment (start 154.1283 78.4236) (end 154.1513 78.4466) (width 1) (layer F.Cu) (net 14))
+  (segment (start 151.3323 78.4236) (end 154.1283 78.4236) (width 1) (layer F.Cu) (net 14))
   (segment (start 139.2923 73.5211) (end 143.1278 73.5211) (width 1) (layer F.Cu) (net 14))
   (segment (start 135.9538 73.5211) (end 135.4823 73.9926) (width 1) (layer F.Cu) (net 14))
@@
   (segment (start 145.6058 73.5211) (end 143.1278 73.5211) (width 1) (layer F.Cu) (net 14))
   (segment (start 151.1033 68.0236) (end 145.6058 73.5211) (width 1) (layer F.Cu) (net 14))
-  (segment (start 151.3323 79.2476) (end 145.6058 73.5211) (width 1) (layer F.Cu) (net 14))
-  (segment (start 151.3323 81.7256) (end 151.3323 79.2476) (width 1) (layer F.Cu) (net 14))
   (segment (start 157.4843 68.0236) (end 157.1993 67.7386) (width 0.5) (layer F.Cu) (net 15))
   (segment (start 166.0893 82.5506) (end 166.0893 78.8186) (width 0.5) (layer F.Cu) (net 15))
@@
   (via (at 152.6273 116.0296) (size 2.4) (drill 1.2) (layers F.Cu B.Cu) (net 18))
   (via (at 139.5463 87.9626) (size 0.8) (drill 0.4) (layers F.Cu B.Cu) (net 1))
+  (segment (start 155.6573 80.8326) (end 155.6753 80.8506) (width 1) (layer F.Cu) (net 7))
+  (segment (start 154.1513 80.8326) (end 155.6573 80.8326) (width 1) (layer F.Cu) (net 7))
+  (segment (start 154.1513 76.3966) (end 155.1583 76.3966) (width 0.5) (layer F.Cu) (net 13))
+  (segment (start 155.1583 76.3966) (end 155.8023 77.0406) (width 0.5) (layer F.Cu) (net 13))
+  (segment (start 155.8023 78.8186) (end 156.9453 79.9616) (width 0.5) (layer F.Cu) (net 13))
+  (segment (start 155.8023 77.0406) (end 155.8023 78.8186) (width 0.5) (layer F.Cu) (net 13))
+  (segment (start 150.5083 78.4236) (end 145.6058 73.5211) (width 1) (layer F.Cu) (net 14))
+  (segment (start 151.3323 78.4236) (end 150.5083 78.4236) (width 1) (layer F.Cu) (net 14))
   (segment (start 161.0093 80.3566) (end 160.6143 79.9616) (width 0.5) (layer F.Cu) (net 19))
   (segment (start 161.0093 82.5506) (end 161.0093 80.3566) (width 0.5) (layer F.Cu) (net 19))
@@
     (polygon
       (pts
-        (xy 195.8073 81.3586) (xy 155.8023 81.3586) (xy 155.8023 87.5816) (xy 143.4833 87.5816) (xy 143.4833 78.9456)
+        (xy 195.8073 81.3586) (xy 155.8023 81.3586) (xy 155.8023 84.7876) (xy 145.5153 84.7876) (xy 145.5153 78.9456)
         (xy 134.3393 78.9456) (xy 134.3393 75.3896) (xy 195.8073 75.3896)
       )
@@
     (polygon
       (pts
-        (xy 195.6803 81.3586) (xy 156.6913 81.3586) (xy 156.6913 87.5816) (xy 148.5633 87.5816) (xy 148.5633 73.2306)
+        (xy 195.6803 81.3586) (xy 156.6913 81.3586) (xy 156.6913 87.4546) (xy 148.5633 87.4546) (xy 148.5633 73.2306)
         (xy 195.6803 73.2306)
       )
@@
     (polygon
       (pts
-        (xy 141.4513 88.7246) (xy 155.1673 88.7246) (xy 155.1673 92.7886) (xy 173.7093 92.7886) (xy 173.7093 100.1546)
-        (xy 134.3393 100.1546) (xy 134.3393 85.4226) (xy 141.4513 85.4226)
+        (xy 141.4513 92.7886) (xy 155.1673 92.7886) (xy 173.7093 92.7886) (xy 173.7093 100.1546) (xy 134.3393 100.1546)
+        (xy 134.3393 85.4226) (xy 141.4513 85.4226)
       )
     )

Commit message: VER2.5
Parts:
- removed R8, R9: 10k, Resistor_SMD:R_0805_2012Metric_Pad1.15x1.40mm_HandSolder
- added C12: 10u, Capacitor_SMD:C_0805_2012Metric_Pad1.15x1.40mm_HandSolder, F.Cu at (155.0, 86.4)
- added C13: 10u, Capacitor_SMD:C_0805_2012Metric_Pad1.15x1.40mm_HandSolder, F.Cu at (154.2, 89.9)
- added U2: LM1117GS-3.3, Package_TO_SOT_SMD:SOT-223, F.Cu at (148.2, 88.7)
- U1: value LM1117-ADJ -> LM1117GS-5.0
- moved R7 6.14 mm to (167.5, 76.5), turned to 180 degrees
- moved C17 1.26 mm to (155.0, 78.4), turned to 0 degrees
Connections:
- R1 pad 1: +5V -> +3V3
Routing:
- net +3V3: track 0.00 -> 24.8 mm, vias 0 -> 2
- net IN-: track 27.6 -> 22.4 mm
- net FLT: track 18.7 -> 15.7 mm
- net RDY: track 16.0 -> 13.3 mm
- net DC-: track 47.8 -> 49.1 mm
- net GNDA: track 47.5 -> 46.3 mm
- net +5V: track 9.88 -> 8.98 mm, vias 3 -> 2
- net +15V_H: vias 3 -> 2
- added copper zone on F.Cu, net GNDA

Commit message: VER2.6
Parts:
- removed D6: LPSR_50-NP, LPSR:LPSR_50
- added C14: 10u, Capacitor_SMD:C_0805_2012Metric_Pad1.18x1.45mm_HandSolder, F.Cu at (187.8, 82.7)
- added C15: 1n, Capacitor_SMD:C_0805_2012Metric_Pad1.18x1.45mm_HandSolder, B.Cu at (188.4, 79.9)
- added C16: 10u, Capacitor_SMD:C_0805_2012Metric_Pad1.18x1.45mm_HandSolder, B.Cu at (176.6, 77.7)
- added R10: 6.2k, Resistor_SMD:R_0805_2012Metric_Pad1.20x1.40mm_HandSolder, F.Cu at (195.6, 73.9)
- added R11: 3к, Resistor_SMD:R_0805_2012Metric_Pad1.20x1.40mm_HandSolder, F.Cu at (195.6, 78.1)
- added R12: 100k, Resistor_SMD:R_0805_2012Metric_Pad1.20x1.40mm_HandSolder, F.Cu at (190.8, 78.1)
- added R13: 300k, Resistor_SMD:R_0805_2012Metric_Pad1.20x1.40mm_HandSolder, B.Cu at (185.0, 76.5)
- added R14: 100k, Resistor_SMD:R_0805_2012Metric_Pad1.20x1.40mm_HandSolder, F.Cu at (193.2, 78.1)
- added R15: 10k, Resistor_SMD:R_0805_2012Metric_Pad1.20x1.40mm_HandSolder, F.Cu at (179.6, 69.1)
- added R16: 13k, Resistor_SMD:R_0805_2012Metric_Pad1.20x1.40mm_HandSolder, F.Cu at (174.4, 68.1)
- added R17: 110, Resistor_SMD:R_0805_2012Metric_Pad1.20x1.40mm_HandSolder, F.Cu at (198.2, 73.9)
- added R18: 110, Resistor_SMD:R_0805_2012Metric_Pad1.20x1.40mm_HandSolder, F.Cu at (200.6, 78.1)
- added R19: 110, Resistor_SMD:R_0805_2012Metric_Pad1.20x1.40mm_HandSolder, F.Cu at (200.6, 73.9)
- added R20: 20k, Resistor_SMD:R_0805_2012Metric_Pad1.20x1.40mm_HandSolder, B.Cu at (187.4, 76.4)
- added R21: 15, Resistor_SMD:R_0805_2012Metric_Pad1.20x1.40mm_HandSolder, F.Cu at (174.4, 64.1)
- added R22: 110, Resistor_SMD:R_0805_2012Metric_Pad1.20x1.40mm_HandSolder, F.Cu at (172.0, 64.1)
- added R8: 0, Diode_SMD:D_SOD-123, F.Cu at (177.8, 96.9)
- added R9: 110, Resistor_SMD:R_0805_2012Metric_Pad1.20x1.40mm_HandSolder, F.Cu at (198.2, 78.1)
- added U3: LMV324, Package_SO:SOIC-14_3.9x8.7mm_P1.27mm, F.Cu at (176.6, 77.7)
- C3: value C_Small -> 1n; footprint Capacitor_SMD:C_0805_2012Metric_Pad1.15x1.40mm_HandSolder -> Capacitor_SMD:C_0805_2012Metric_Pad1.18x1.45mm_HandSolder
- D3: value MMSZ5223B -> NSM2011; footprint Diode_SMD:D_SOD-123 -> Package_SO:SOIC-16W_7.5x10.3mm_P1.27mm; moved to B.Cu
- R3: value R_Small -> 360; footprint Resistor_SMD:R_0805_2012Metric_Pad1.15x1.40mm_HandSolder -> Resistor_SMD:R_0805_2012Metric_Pad1.20x1.40mm_HandSolder
- R4: value 6.8k -> 12k
- moved C3 26.3 mm to (168.2, 67.3), turned to -90 degrees
- moved D3 13.9 mm to (187.8, 87.3)
- moved R3 3.80 mm to (193.2, 73.9), turned to -90 degrees
Connections:
- D3 pad 1: Net-(D3-Pad1) -> OUT-
- D3 pad 2: Net-(D3-Pad2) -> OUT-
- D5 pad 2: Net-(D3-Pad2) -> Net-(D5-Pad2)
- R3 pad 2: Measure -> +5V
- R4 pad 2: Net-(D3-Pad1) -> Net-(R4-Pad2)
Routing:
- net Net-(R12-Pad2): track 0.00 -> 30.3 mm, vias 0 -> 1
- net Net-(D3-Pad1): track 22.6 -> 0.00 mm, vias 2 -> 0
- net Net-(R4-Pad2): track 0.00 -> 22.5 mm, vias 0 -> 2
- net Measure: track 46.2 -> 28.0 mm, vias 1 -> 0
- net GNDA: track 46.3 -> 62.8 mm, vias 4 -> 10
- net Net-(R15-Pad2): track 0.00 -> 14.8 mm
- net Net-(D5-Pad2): track 0.00 -> 13.1 mm
- net Net-(D3-Pad2): track 13.1 -> 0.00 mm
- net +5V: track 8.98 -> 17.4 mm, vias 2 -> 5
- net VOUT: track 0.00 -> 5.30 mm
- net Net-(R14-Pad1): track 0.00 -> 4.60 mm
- net Net-(R10-Pad2): track 6.66 -> 2.40 mm
- net Net-(R16-Pad1): track 0.00 -> 3.81 mm
- net Net-(R11-Pad2): track 0.00 -> 2.60 mm
- net Net-(R13-Pad1): track 0.00 -> 2.42 mm
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- added copper zone on B.Cu, net OUT-
Other:
- outline, holes or cut-outs redrawn
- net class Default removed
