File: Драйвер IGBT/Драйвер IGBT.sch (KiCad schematic (older format))
At the start: 41 parts, among them J1 DC+, J2 DC-, J3 Control Connector, J4 OUT-, J5 OUT+, Q1 HGTG20N60A4, U3 L78L05ACUTR

Commit message: VER2.0
Parts:
- removed D1: VS-60APU06PBF, Package_TO_SOT_THT:TO-247-3_Vertical, symbol Diode_My:Diode_AKA
- removed D7: LED_FLT, LED_SMD:LED_0603_1608Metric_Pad1.05x0.95mm_HandSolder, symbol Device:LED_Small
- removed U3: L78L05ACUTR, Package_TO_SOT_SMD:SOT-89-3, symbol Regulator_Linear:LM78M05_TO220
- added D1: VS-60EPF06-M3, Package_TO_SOT_THT:TO-247-2_Vertical, symbol Device:D
- added R8, R9: 10k, Resistor_SMD:R_0805_2012Metric_Pad1.15x1.40mm_HandSolder, symbol Device:R_Small
- added U1: LM1117-ADJ, Package_TO_SOT_SMD:SOT-223, symbol Regulator_Linear:LM1117-ADJ
- C17: value 0.33u -> 10u
- C18: value 0.1u -> 10u
- D8: footprint Converter_DCDC:Converter_DCDC_TRACO_TMR-1-xxxx_Dual_THT -> TRACO:TMA1515S
Connections:
- net labels added: DC+
- no-connect marks 3 -> 2
Other:
- moved on the sheet: Q1, R2

Commit message: VER2.4
Parts:
- removed R8, R9: 10k, Resistor_SMD:R_0805_2012Metric_Pad1.15x1.40mm_HandSolder, symbol Device:R_Small
- added C12, C13: 10u, Capacitor_SMD:C_0805_2012Metric_Pad1.15x1.40mm_HandSolder, symbol Device:C_Small
- added U2: LM1117GS-3.3, Package_TO_SOT_SMD:SOT-223, symbol Regulator_Linear:LM1117-ADJ
- U1: value LM1117-ADJ -> LM1117GS-5.0
Connections:
- net labels added: +3.3V
- wire segments 59 -> 67
Other:
- moved on the sheet: C1, C11, C4, C5, C8, D1, Q1, R2

Commit message: VER2.6
Parts:
- removed D3: MMSZ5223B, Diode_SMD:D_SOD-123, symbol Device:D_Zener_Small
- removed D8: TMA1515S, TRACO:TMA1515S, symbol Linear~Regulator:TMA1515S
- added D8: TMA1515S, TRACO:TMA1515S, symbol Linear_Regulator:TMA1515S
- added R8: 0, Diode_SMD:D_SOD-123, symbol Device:R_Small
- C3: value C_Small -> 1u
- D2: symbol Драйвер-IGBT-rescue:ISO54-Driver-Driver_SiC-rescue-Драйвер-IGBT-rescue -> Драйвер-IGBT-rescue:ISO54-Driver-Driver_SiC-rescue-Драйвер-IGBT-rescue-Драйвер-IGBT-rescue
- D6: symbol Драйвер-IGBT-rescue:LPSR_50-NP-LPSR-cache-Драйвер-IGBT-rescue -> Драйвер-IGBT-rescue:LPSR_50-NP-LPSR-cache-Драйвер-IGBT-rescue-Драйвер-IGBT-rescue
- R3: value R_Small -> 200
- R4: value 6.8k -> 12k
Other:
- note added: "Зарицкий"
- moved on the sheet: C1, C10, C11, C2, C3, C4, C5, C6, C7, C8, C9, D1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
